Commit message: making improvements to agent in sim

File: source/isaaclab_tasks/isaaclab_tasks/direct/crazyflie_l2f/assets/crazyflie_21.urdf (robot description, URDF)
Before this commit: robot crazyflie_21, 9 links, 8 joints
Links:
- link arm1: geometry visual box size=0.04 0.003 0.0015
- link arm2: geometry visual box size=0.04 0.003 0.0015
- link arm3: geometry visual box size=0.04 0.003 0.0015
- link arm4: geometry visual box size=0.04 0.003 0.0015
- link body: geometry collision box size=0.03 0.03 0.012; visual box size=0.028 0.028 0.008
- link m1_prop: geometry visual cylinder length=0.003 radius=0.0225
- link m2_prop: geometry visual cylinder length=0.003 radius=0.0225
- link m3_prop: geometry visual cylinder length=0.003 radius=0.0225
- link m4_prop: geometry visual cylinder length=0.003 radius=0.0225
